File: xmachine.sch (EAGLE design)
At the start: 2 parts, among them IC1 ECP5-LFE5U-XXF-8BG381C, J1 PDS-030

Commit message: added level shifters and flash memory
Parts:
- added IC2, IC3, IC4, IC5, IC6, IC7, IC8: SN74LVC16T245, sk9k-Texas Instruments:SN74LVC16T245
- added IC9: IS25WP128-JBLE, sk9k-Memory:W25Q64FWSSIG
- added R1, R2, R3, R4: 10k, sk9k-RCL:RESISTOR0402-RES
- added R5: 1k, sk9k-RCL:RESISTOR0402-RES
- added R6: 4.7k, sk9k-RCL:RESISTOR0402-RES
Connections:
- new net /BG: IC6.1B1, J1G$2./BG
- new net /BGACK: IC7.1B2, J1G$2./BGACK
- new net /BR: IC7.1B1, J1G$2./BR
- new net /BUSLOCK: IC7.1B7, J1G$2./BUSLOCK
- new net /CBACK: IC7.1B4, J1G$2./CBACK
- new net /CBREQ: IC6.1B2, J1G$2./CBREQ
- new net /CIOUT: IC6.1B3, J1G$2./CIOUT
- new net /IRQ1: J1G$2./IRQ1
- new net /IRQ2: J1G$2./IRQ2
- new net /IRQ3: J1G$2./IRQ3
- new net /NUBUS: IC6.1B5, J1G$2./NUBUS
- new net /RMC: IC6.1B4, J1G$2./RMC
- new net /STERM: IC7.1B3, J1G$2./STERM
- new net /TM0A: IC7.1B5, J1G$2./TM0A
- new net /TM1A: IC7.1B6, J1G$2./TM1A
- new net 3V3: IC2.VCCA, IC3.VCCA, IC4.VCCA, IC5.VCCA, IC6.VCCA, IC7.1DIR, IC7.2DIR, IC7.VCCA, IC9.VCC, R1.2, R2.2, R3.2, R4.2, R5.2, R6.2
- new net 5V: IC2.VCCB, IC3.VCCB, IC4.VCCB, IC5.VCCB, IC6.VCCB, IC7.VCCB, J1G$2.5V
- new net A0: IC2.1B1, J1G$1.A0
- new net A1: IC2.1B2, J1G$1.A1
- new net A10: IC2.2B3, J1G$1.A10
- new net A11: IC2.2B4, J1G$1.A11
- new net A12: IC2.2B5, J1G$1.A12
- new net A13: IC2.2B6, J1G$1.A13
- new net A14: IC2.2B7, J1G$1.A14
- new net A15: IC2.2B8, J1G$1.A15
- new net A16: IC3.1B1, J1G$1.A16
- new net A17: IC3.1B2, J1G$1.A17
- new net A18: IC3.1B3, J1G$1.A18
- new net A19: IC3.1B4, J1G$1.A19
- new net A2: IC2.1B3, J1G$1.A2
- new net A20: IC3.1B5, J1G$1.A20
- new net A21: IC3.1B6, J1G$1.A21
- new net A22: IC3.1B7, J1G$1.A22
- new net A23: IC3.1B8, J1G$1.A23
- new net A24: IC3.2B1, J1G$1.A24
- new net A25: IC3.2B2, J1G$1.A25
- new net A26: IC3.2B3, J1G$1.A26
- new net A27: IC3.2B4, J1G$1.A27
- new net A28: IC3.2B5, J1G$1.A28
- new net A29: IC3.2B6, J1G$1.A29
- new net A3: IC2.1B4, J1G$1.A3
- new net A30: IC3.2B7, J1G$1.A30
- new net A31: IC3.2B8, J1G$1.A31
- new net A4: IC2.1B5, J1G$1.A4
- new net A5: IC2.1B6, J1G$1.A5
- new net A6: IC2.1B7, J1G$1.A6
- new net A7: IC2.1B8, J1G$1.A7
- new net A8: IC2.2B1, J1G$1.A8
- new net A9: IC2.2B2, J1G$1.A9
- new net ADDR_DIR: IC2.1DIR, IC2.2DIR, IC3.1DIR, IC3.2DIR
- new net C16M: IC6.2B1, J1G$2.C16M
- new net CPUCLK: IC6.1B7, J1G$2.CPUCLK
- new net DATA_DIR: IC4.1DIR, IC4.2DIR, IC5.1DIR, IC5.2DIR
- new net ECLK: IC6.1B8, J1G$2.ECLK
- new net FLASH_CLK: IC9.CLK, R5.1
- new net FLASH_CS: IC9.CS, R6.1
- new net FLASH_HOLD: IC9.HOLD/IO3, R2.1
- new net FLASH_MISO: IC9.SO/IO1, R3.1
- new net FLASH_MOSI: IC9.SI/IO0, R4.1
- new net FLASH_WP: IC9.WP/IO2, R1.1
- new net GND: IC2.1OE, IC2.2OE, IC2.GND, IC3.1OE, IC3.2OE, IC3.GND, IC4.1OE, IC4.2OE, IC4.GND, IC5.1OE, IC5.2OE, IC5.GND, IC6.1DIR, IC6.1OE, IC6.2DIR, IC6.GND, IC7.1OE, IC7.2OE, IC7.GND, IC9.GND, J1G$2.GND
- new net N$100: IC2.1A4
- new net N$101: J1G$2.RES1
- new net N$102: J1G$2.RES2
- new net N$103: J1G$2.RES3
- new net N$107: J1G$2./IPL0
- new net N$110: J1G$2./R/W
- new net N$111: J1G$2./AS
- new net N$113: IC2.1A5
- new net N$114: IC2.1A6
- new net N$115: IC2.1A7
- new net N$116: IC2.1A8
- new net N$118: IC2.2A1
- new net N$119: IC2.2A2
- new net N$120: IC2.2A3
- new net N$122: IC2.2A4
- new net N$123: IC2.2A5
- new net N$124: IC2.2A6
- new net N$125: IC2.2A7
- new net N$126: IC2.2A8
- new net N$150: IC3.1A1
- new net N$151: IC3.1A2
- new net N$152: IC3.1A3
- new net N$153: IC3.1A4
- new net N$154: IC3.1A5
- new net N$155: IC3.1A6
- new net N$156: IC3.1A7
- new net N$157: IC3.1A8
- new net N$159: IC3.2A1
- new net N$160: IC3.2A2
- new net N$162: IC3.2A3
- new net N$163: IC3.2A4
- new net N$164: IC3.2A5
- new net N$165: IC3.2A6
- new net N$166: IC3.2A7
- new net N$167: IC3.2A8
- new net N$190: IC5.1B1
- new net N$191: IC5.1B2
- new net N$192: IC5.1B3
- new net N$193: IC5.1B4
- new net N$194: IC5.1B5
- new net N$195: IC5.1B6
- new net N$196: IC5.1B7
- new net N$197: IC5.1B8
- new net N$199: IC5.2B1
- new net N$200: IC5.2B2
- new net N$202: IC5.2B3
- new net N$203: IC5.2B4
- new net N$204: IC5.2B5
- new net N$205: IC5.2B6
- new net N$206: IC5.2B7
- new net N$207: IC5.2B8
- new net N$209: IC5.1A1
- new net N$210: IC5.1A2
- new net N$211: IC5.1A3
- new net N$212: IC5.1A4
- new net N$213: IC5.1A5
- new net N$214: IC5.1A6
- new net N$215: IC5.1A7
- new net N$216: IC5.1A8
- new net N$218: IC5.2A1
- new net N$219: IC5.2A2
- new net N$220: IC5.2A3
- new net N$222: IC5.2A4
- new net N$223: IC5.2A5
- new net N$224: IC5.2A6
- new net N$225: IC5.2A7
- new net N$226: IC5.2A8
- new net N$229: IC4.1A1
- new net N$230: IC4.1A2
- new net N$231: IC4.1A3
- new net N$232: IC4.1A4
- new net N$233: IC4.1A5
- new net N$234: IC4.1A6
- new net N$235: IC4.1A7
- new net N$236: IC4.1A8
- new net N$238: IC4.2A1
- new net N$239: IC4.2A2
- new net N$240: IC4.2A3
- new net N$242: IC4.2A4
- new net N$243: IC4.2A5
- new net N$244: IC4.2A6
- new net N$245: IC4.2A7
- new net N$246: IC4.2A8
- new net N$250: IC4.1B1
- new net N$251: IC4.1B2
- new net N$252: IC4.1B3
- new net N$253: IC4.1B4
- new net N$254: IC4.1B5
- new net N$255: IC4.1B6
- new net N$256: IC4.1B7
- new net N$257: IC4.1B8
- new net N$259: IC4.2B1
- new net N$260: IC4.2B2
- new net N$262: IC4.2B3
- new net N$263: IC4.2B4
- new net N$264: IC4.2B5
- new net N$265: IC4.2B6
- new net N$266: IC4.2B7
- new net N$267: IC4.2B8
- new net N$270: IC6.1A1
- new net N$271: IC6.1A2
- new net N$272: IC6.1A3
- new net N$273: IC6.1A4
- new net N$274: IC6.1A5
- new net N$275: IC6.1A6
- new net N$276: IC6.1A7
- new net N$277: IC6.1A8
- new net N$279: IC6.2A1
- new net N$280: IC6.2A2
- new net N$282: IC6.2A3
- new net N$283: IC6.2A4
- new net N$284: IC6.2A5
- new net N$285: IC6.2A6
- new net N$286: IC6.2A7
- new net N$287: IC6.2A8
- new net N$298: IC6.2OE
- new net N$307: IC7.1B8
- new net N$309: IC7.1A1
- new net N$310: IC7.1A2
- new net N$311: IC7.1A3
- new net N$312: IC7.1A4
- new net N$313: IC7.1A5
- new net N$314: IC7.1A6
- new net N$315: IC7.1A7
- new net N$316: IC7.1A8
- new net N$318: IC7.2A1
- new net N$319: IC7.2A2
- new net N$320: IC7.2A3
- new net N$322: IC7.2A4
- new net N$323: IC7.2A5
- new net N$324: IC7.2A6
- new net N$325: IC7.2A7
- new net N$326: IC7.2A8
- new net N$339: IC7.2B1
- new net N$340: IC7.2B2
- new net N$342: IC7.2B3
- new net N$343: IC7.2B4
- new net N$344: IC7.2B5
- new net N$345: IC7.2B6
- new net N$346: IC7.2B7
- new net N$347: IC7.2B8
- new net N$348: IC8.1DIR
- new net N$349: IC8.1A1
- new net N$35: J1G$2./IPL2
- new net N$350: IC8.1A2
- new net N$351: IC8.1A3
- new net N$352: IC8.1A4
- new net N$353: IC8.1A5
- new net N$354: IC8.1A6
- new net N$355: IC8.1A7
- new net N$356: IC8.1A8
- new net N$357: IC8.2DIR
- new net N$358: IC8.2A1
- new net N$359: IC8.2A2
- new net N$360: IC8.2A3
- new net N$362: IC8.2A4
- new net N$363: IC8.2A5
- new net N$364: IC8.2A6
- new net N$365: IC8.2A7
- new net N$366: IC8.2A8
- new net N$367: IC8.GND
- new net N$368: IC8.VCCB
- new net N$369: IC8.1OE
- new net N$370: IC8.1B1
- new net N$371: IC8.1B2
- new net N$372: IC8.1B3
- new net N$373: IC8.1B4
- new net N$374: IC8.1B5
- new net N$375: IC8.1B6
- new net N$376: IC8.1B7
- new net N$377: IC8.1B8
- new net N$378: IC8.2OE
- new net N$379: IC8.2B1
- new net N$38: J1G$2./DSACK1
- new net N$380: IC8.2B2
- new net N$382: IC8.2B3
- new net N$383: IC8.2B4
- new net N$384: IC8.2B5
- new net N$385: IC8.2B6
- new net N$386: IC8.2B7
- new net N$387: IC8.2B8
- new net N$4: IC6.2B4
- new net N$40: J1G$1.D0
- new net N$41: J1G$1.D1
- new net N$42: J1G$1.D2
- new net N$43: J1G$1.D3
- new net N$44: J1G$1.D4
- new net N$45: J1G$1.D5
- new net N$46: J1G$1.D6
- new net N$47: J1G$1.D7
- new net N$48: J1G$1.D8
- new net N$49: J1G$1.D9
- new net N$5: IC6.2B5
- new net N$50: J1G$1.D10
- new net N$51: J1G$1.D11
- new net N$52: J1G$1.D12
- new net N$53: J1G$1.D13
- new net N$54: J1G$1.D14
- new net N$55: J1G$1.D15
- new net N$56: J1G$1.D16
- new net N$57: J1G$1.D17
- new net N$58: J1G$1.D18
- new net N$59: J1G$1.D19
- new net N$6: IC6.2B6
- new net N$60: J1G$1.D20
- new net N$61: J1G$1.D21
- new net N$62: J1G$1.D22
- new net N$63: J1G$1.D23
- new net N$64: J1G$1.D24
- new net N$65: J1G$1.D25
- new net N$66: J1G$1.D26
- new net N$67: J1G$1.D27
- new net N$68: J1G$1.D28
- new net N$69: J1G$1.D29
- new net N$7: IC6.2B7
- new net N$70: J1G$1.D30
- new net N$71: J1G$1.D31
- new net N$73: J1G$2.FC2
- new net N$74: J1G$2./RESET
- new net N$78: J1G$2./IPL1
- new net N$79: J1G$2./DS
- new net N$8: IC6.2B8
- new net N$81: J1G$2./DSACK0
- new net N$84: J1G$2.FC1
- new net N$85: J1G$2./BERR
- new net N$89: IC2.1A1
- new net N$90: IC2.1A2
- new net N$91: J1G$2.FC0
- new net N$92: J1G$2./HALT
- new net N$94: IC2.1A3
- new net N$96: J1G$2.-5V
- new net N$97: J1G$2.12V
- new net N$98: J1G$2.-12V
- new net POWEROFF: IC6.1B6
- new net PWROFF: J1G$2.PWROFF
- new net SIZ0: J1G$2.SIZ0
- new net SIZ1: J1G$2.SIZ1
Other:
- note added: "inputs to 030"
- note added: "outputs from 030"
